Commit message: Update Lidar

File: skratch_description/description/sensor_mounts/lidar_mount.xacro (robot description, xacro)
@@ -34,5 +34,5 @@
         </joint>
         <xacro:hokuyo_urg_lidar name="${name}_hokuyo_urg_lidar" parent="${name}_lidar_mount">
-            <origin xyz="0.045 -0.045 -0.095" rpy="3.14 0.0 -0.77"/>
+            <origin xyz="0.045 -0.045 -0.1" rpy="3.14 0.0 -0.77"/>
         </xacro:hokuyo_urg_lidar>
     </xacro:macro>

File: skratch_description/description/sensors/hokuyo_urg_04lx_ug01.xacro (robot description, xacro)
@@ -24,6 +24,35 @@
             </collision>
         </link>
-        <gazebo reference="${name}">
+        <gazebo reference="${name}_hokuyo_urg_lidar_link">
             <material>Gazebo/Black</material>
+            <sensor type="gpu_lidar" name="${name}_hokuyo_urg_lidar">
+                <pose>0 0 0.06 0 0 0</pose>
+                <visualize>true</visualize>
+                <update_rate>10</update_rate>
+                <lidar>
+                    <scan>
+                        <horizontal>
+                            <samples>682</samples>
+                            <resolution>1</resolution>
+                            <min_angle>-2.35619449</min_angle>
+                            <!-- -135° in rad -->
+                            <max_angle>2.35619449</max_angle>
+                            <!-- 135° in rad -->
+                        </horizontal>
+                    </scan>
+                    <range>
+                        <min>0.06</min>
+                        <max>5.6</max>
+                        <resolution>0.001</resolution>
+                    </range>
+                    <noise>
+                        <type>gaussian</type>
+                        <mean>0.0</mean>
+                        <stddev>0.005</stddev>
+                    </noise>
+                </lidar>
+                <topic>/${name}_scan</topic>
+                <gz_frame_id>hokuyo_urg04lx_link</gz_frame_id>
+            </sensor>
         </gazebo>
         <joint name="${name}_hokuyo_urg_lidar_mount_joint" type="fixed">
