Commit message: Add Licence

File: skratch_description/description/base/kinova_arm_base_plate.xacro (robot description, xacro)
@@ -1,3 +1,10 @@
 <?xml version="1.0"?>
+<!--
+Copyright (c) 2025
+b-it-bots
+Hochschule Bonn-Rhein-Sieg
+Authors:
+Chaitanya Gumudala
+-->
 <robot name="arm_base_plate" xmlns:xacro="http://www.ros.org/wiki/xacro">
     <xacro:macro name="arm_base_plate" params="name">

File: skratch_description/description/base/skratch_base.xacro (robot description, xacro)
@@ -1,3 +1,10 @@
 <?xml version="1.0"?>
+<!--
+Copyright (c) 2025
+b-it-bots
+Hochschule Bonn-Rhein-Sieg
+Authors:
+Chaitanya Gumudala
+-->
 <robot name="skratch_base" xmlns:xacro="http://www.ros.org/wiki/xacro">
     <xacro:macro name="skratch_base" params="name">

File: skratch_description/description/sensor_mounts/lidar_mount.xacro (robot description, xacro)
@@ -1,3 +1,10 @@
 <?xml version="1.0"?>
+<!--
+Copyright (c) 2025
+b-it-bots
+Hochschule Bonn-Rhein-Sieg
+Authors:
+Chaitanya Gumudala
+-->
 <robot name="lidar_mount" xmlns:xacro="http://www.ros.org/wiki/xacro">
     <xacro:macro name="lidar_mount" params="name parent *origin">

File: skratch_description/description/sensors/hokuyo_urg_04lx_ug01.xacro (robot description, xacro)
@@ -1,3 +1,10 @@
 <?xml version="1.0"?>
+<!--
+Copyright (c) 2025
+b-it-bots
+Hochschule Bonn-Rhein-Sieg
+Authors:
+Chaitanya Gumudala
+-->
 <robot name="hokuyo_urg_lidar" xmlns:xacro="http://www.ros.org/wiki/xacro">
     <xacro:macro name="hokuyo_urg_lidar" params="name parent *origin">

File: skratch_description/description/skratch.urdf.xacro (robot description, xacro)
@@ -1,4 +1,12 @@
 <?xml version="1.0" ?>
+<!--
+Copyright (c) 2025
+b-it-bots
+Hochschule Bonn-Rhein-Sieg
+Authors:
+Chaitanya Gumudala
+-->
 <robot name="skratch" xmlns:xacro="http://www.ros.org/wiki/xacro">
+    <xacro:arg name="movable_joints" default="true"/>
     <xacro:include filename="$(find skratch_description)/description/base/skratch_base.xacro"/>
     <xacro:include filename="$(find skratch_description)/description/base/kinova_arm_base_plate.xacro"/>
@@ -6,5 +14,5 @@
     <xacro:include filename="$(find skratch_description)/description/skratch_ros.xacro"/>
     <xacro:include filename="$(find skratch_description)/description/sensor_mounts/lidar_mount.xacro"/>
-    <xacro:include filename="$(find kinova_arm_description)/description/kinova_arm.xacro"/>
+    <!-- <xacro:include filename="$(find kinova_arm_description)/description/kinova_arm.xacro"/> -->
     <link name="base_link"/>
     <xacro:skratch_base name="skratch_base"/>
@@ -14,14 +22,14 @@
         <child link="skratch_base"/>
     </joint>
-    <xacro:kelo_drive_top_part name="front_left_drive_top_part" parent="skratch_base" drive_name="skratch_1_drive">
+    <xacro:kelo_drive_top_part name="front_left_drive_top_part" parent="skratch_base" drive_name="skratch_1_drive" movable_joints="$(arg movable_joints)">
         <origin xyz="0.202 0.118 -0.054" rpy="0.0 0 0.0"/>
     </xacro:kelo_drive_top_part>
-    <xacro:kelo_drive_top_part name="front_right_drive_top_part" parent="skratch_base" drive_name="skratch_2_drive">
+    <xacro:kelo_drive_top_part name="front_right_drive_top_part" parent="skratch_base" drive_name="skratch_2_drive" movable_joints="$(arg movable_joints)">
         <origin xyz="0.202 -0.118 -0.054" rpy="0.0 0 0.0"/>
     </xacro:kelo_drive_top_part>
-    <xacro:kelo_drive_top_part name="rear_left_drive_top_part" parent="skratch_base" drive_name="skratch_3_drive">
+    <xacro:kelo_drive_top_part name="rear_left_drive_top_part" parent="skratch_base" drive_name="skratch_3_drive" movable_joints="$(arg movable_joints)">
         <origin xyz="-0.202  0.118 -0.054" rpy="0.0 0 0.0"/>
     </xacro:kelo_drive_top_part>
-    <xacro:kelo_drive_top_part name="rear_right_drive_top_part" parent="skratch_base" drive_name="skratch_4_drive">
+    <xacro:kelo_drive_top_part name="rear_right_drive_top_part" parent="skratch_base" drive_name="skratch_4_drive" movable_joints="$(arg movable_joints)">
         <origin xyz="-0.202 -0.118 -0.054" rpy="0.0 0 0.0"/>
     </xacro:kelo_drive_top_part>
@@ -38,9 +46,9 @@
         <origin xyz="-0.272 0.168 0.0025" rpy="0.0 0.0 3.14"/>
     </xacro:lidar_mount>
-    <xacro:kinova_arm/>
-    <joint name="kinova_arm_joint" type="fixed">
+    <!-- <xacro:kinova_arm/> -->
+    <!-- <joint name="kinova_arm_joint" type="fixed">
         <origin xyz="0.0 0.0 0.02" rpy="0 0 0"/>
         <parent link="arm_base_plate"/>
         <child link="kinova_base"/>
-    </joint>
+    </joint> -->
 </robot>

File: skratch_description/description/skratch_ros.xacro (robot description, xacro)
@@ -1,3 +1,10 @@
 <?xml version="1.0"?>
+<!--
+Copyright (c) 2025
+b-it-bots
+Hochschule Bonn-Rhein-Sieg
+Authors:
+Chaitanya Gumudala
+-->
 <robot xmlns:xacro="http://www.ros.org/wiki/xacro">
     <xacro:macro name="joint_interface" params="joint_name">

File: skratch_description/description/wheels/kelo_drive.xacro (robot description, xacro)
@@ -1,5 +1,36 @@
 <?xml version="1.0"?>
+<!--
+Copyright (c) 2021
+KELO Robotics GmbH
+Author:
+Sushant Chavan
+Maintainer:
+Chaitanya Gumudala
+This software is published under a dual-license: GNU Lesser General Public
+License LGPL 2.1 and BSD license. The dual-license implies that users of this
+code may choose which terms they prefer.
+Redistribution and use in source and binary forms, with or without
+modification, are permitted provided that the following conditions are met:
+* Redistributions of source code must retain the above copyright
+notice, this list of conditions and the following disclaimer.
+* Redistributions in binary form must reproduce the above copyright
+notice, this list of conditions and the following disclaimer in the
+documentation and/or other materials provided with the distribution.
+* Neither the name of Locomotec nor the names of its
+contributors may be used to endorse or promote products derived from
+this software without specific prior written permission.
+This program is free software: you can redistribute it and/or modify
+it under the terms of the GNU Lesser General Public License LGPL as
+published by the Free Software Foundation, either version 2.1 of the
+License, or (at your option) any later version or the BSD license.
+This program is distributed in the hope that it will be useful,
+but WITHOUT ANY WARRANTY; without even the implied warranty of
+MERCHANTABILITY or FITNESS FOR A PARTICULAR PURPOSE. See the
+GNU Lesser General Public License LGPL and the BSD license for more details.
+You should have received a copy of the GNU Lesser General Public
+License LGPL and BSD license along with this program.
+-->
 <robot xmlns:xacro="http://www.ros.org/wiki/xacro">
-    <xacro:macro name="kelo_drive" params="name parent *origin">
+    <xacro:macro name="kelo_drive" params="name parent *origin movable_joints:=true">
         <xacro:include filename="$(find skratch_description)/description/wheels/kelo_drive_wheel.xacro"/>
         <link name="${name}_pivot_link">
@@ -25,18 +56,37 @@
             </inertial>
         </link>
-        <joint name="${name}_pivot_joint" type="continuous">
-            <xacro:insert_block name="origin" />
-            <axis xyz="0 0 1"/>
-            <parent link="${parent}"/>
-            <child link="${name}_pivot_link" />
-            <dynamics damping="0.1" friction="0.05"/>
-            <limit effort="2.0" velocity="1.0"/>
-        </joint>
+        <xacro:if value="${movable_joints}">
+            <joint name="${name}_pivot_joint" type="continuous">
+                <xacro:insert_block name="origin" />
+                <axis xyz="0 0 1"/>
+                <parent link="${parent}"/>
+                <child link="${name}_pivot_link" />
+                <dynamics damping="0.1" friction="0.05"/>
+                <limit effort="2.0" velocity="1.0"/>
+            </joint>
+            <transmission name="${name}_pivot_transmission">
+                <type>transmission_interface/SimpleTransmission</type>
+                <joint name="${name}_pivot_joint">
+                    <hardwareInterface>hardware_interface/EffortJointInterface</hardwareInterface>
+                </joint>
+                <actuator name="${name}_pivot_motor">
+                    <hardwareInterface>hardware_interface/EffortJointInterface</hardwareInterface>
+                    <mechanicalReduction>1</mechanicalReduction>
+                </actuator>
+            </transmission>
+        </xacro:if>
+        <xacro:unless value ="${movable_joints}">
+            <joint name="${name}_pivot_joint" type="fixed">
+                <xacro:insert_block name="origin" />
+                <parent link="${parent}"/>
+                <child link="${name}_pivot_link" />
+            </joint>
+        </xacro:unless>
         <!-- LEFT HUB WHEEL -->
-        <xacro:kelo_drive_wheel name="${name}_left_hub_wheel" parent="${name}_pivot_link">
+        <xacro:kelo_drive_wheel name="${name}_left_hub_wheel" parent="${name}_pivot_link" movable_joints="${movable_joints}">
             <origin xyz="-0.0 0.039326 0.001514" rpy="0 0 0.0"/>
         </xacro:kelo_drive_wheel>
         <!-- RIGHT HUB WHEEL -->
-        <xacro:kelo_drive_wheel name="${name}_right_hub_wheel" parent="${name}_pivot_link">
+        <xacro:kelo_drive_wheel name="${name}_right_hub_wheel" parent="${name}_pivot_link" movable_joints="${movable_joints}">
             <origin xyz="-0.0 -0.039326 0.001514" rpy="0 0 0.0"/>
         </xacro:kelo_drive_wheel>

File: skratch_description/description/wheels/kelo_drive_top_part.xacro (robot description, xacro)
@@ -1,5 +1,12 @@
 <?xml version="1.0"?>
+<!--
+Copyright (c) 2025
+b-it-bots
+Hochschule Bonn-Rhein-Sieg
+Authors:
+Chaitanya Gumudala
+-->
 <robot xmlns:xacro="http://www.ros.org/wiki/xacro">
-    <xacro:macro name="kelo_drive_top_part" params="name parent drive_name:=default_drive_name *origin">
+    <xacro:macro name="kelo_drive_top_part" params="name parent drive_name:=default_drive_name *origin movable_joints:=true">
         <xacro:include filename="$(find skratch_description)/description/wheels/kelo_drive.xacro" />
         <link name="${name}_drive_top_part">
@@ -30,5 +37,5 @@
             <child link="${name}_drive_top_part"/>
         </joint>
-        <xacro:kelo_drive name="${drive_name}" parent="${name}_drive_top_part">
+        <xacro:kelo_drive name="${drive_name}" parent="${name}_drive_top_part" movable_joints="${movable_joints}">
             <origin xyz="0 0 -0.09" rpy="0 0 0.0"/>
         </xacro:kelo_drive>

File: skratch_description/description/wheels/kelo_drive_wheel.xacro (robot description, xacro)
@@ -1,5 +1,36 @@
 <?xml version="1.0"?>
+<!--
+Copyright (c) 2021
+KELO Robotics GmbH
+Author:
+Sushant Chavan
+Maintainer:
+Chaitanya Gumudala
+This software is published under a dual-license: GNU Lesser General Public
+License LGPL 2.1 and BSD license. The dual-license implies that users of this
+code may choose which terms they prefer.
+Redistribution and use in source and binary forms, with or without
+modification, are permitted provided that the following conditions are met:
+* Redistributions of source code must retain the above copyright
+notice, this list of conditions and the following disclaimer.
+* Redistributions in binary form must reproduce the above copyright
+notice, this list of conditions and the following disclaimer in the
+documentation and/or other materials provided with the distribution.
+* Neither the name of Locomotec nor the names of its
+contributors may be used to endorse or promote products derived from
+this software without specific prior written permission.
+This program is free software: you can redistribute it and/or modify
+it under the terms of the GNU Lesser General Public License LGPL as
+published by the Free Software Foundation, either version 2.1 of the
+License, or (at your option) any later version or the BSD license.
+This program is distributed in the hope that it will be useful,
+but WITHOUT ANY WARRANTY; without even the implied warranty of
+MERCHANTABILITY or FITNESS FOR A PARTICULAR PURPOSE. See the
+GNU Lesser General Public License LGPL and the BSD license for more details.
+You should have received a copy of the GNU Lesser General Public
+License LGPL and BSD license along with this program.
+-->
 <robot xmlns:xacro="http://www.ros.org/wiki/xacro">
-    <xacro:macro name="kelo_drive_wheel" params="name parent *origin">
+    <xacro:macro name="kelo_drive_wheel" params="name parent *origin movable_joints:=true">
         <link name="${name}_link">
             <visual>
@@ -27,10 +58,29 @@
             <material>Gazebo/Black</material>
         </gazebo>
-        <joint name="${name}_joint" type="continuous">
-            <xacro:insert_block name="origin" />
-            <axis xyz="0 1 0"/>
-            <parent link="${parent}"/>
-            <child link="${name}_link" />
-        </joint>
+        <xacro:if value="${movable_joints}">
+            <joint name="${name}_joint" type="continuous">
+                <xacro:insert_block name="origin" />
+                <axis xyz="0 1 0"/>
+                <parent link="${parent}"/>
+                <child link="${name}_link" />
+            </joint>
+            <transmission name="${name}_transmission">
+                <type>transmission_interface/SimpleTransmission</type>
+                <joint name="${name}_joint">
+                    <hardwareInterface>hardware_interface/EffortJointInterface</hardwareInterface>
+                </joint>
+                <actuator name="${name}_motor">
+                    <hardwareInterface>hardware_interface/EffortJointInterface</hardwareInterface>
+                    <mechanicalReduction>1</mechanicalReduction>
+                </actuator>
+            </transmission>
+        </xacro:if>
+        <xacro:unless value="${movable_joints}">
+            <joint name="${name}_joint" type="fixed">
+                <xacro:insert_block name="origin" />
+                <parent link="${parent}"/>
+                <child link="${name}_link" />
+            </joint>
+        </xacro:unless>
     </xacro:macro>
 </robot>
