Commit message: Update Dynamics of Pivot

File: skratch_description/description/wheels/kelo_drive.xacro (robot description, xacro)
@@ -62,5 +62,5 @@
                 <parent link="${parent}"/>
                 <child link="${name}_pivot_link" />
-                <dynamics damping="0.1" friction="0.05"/>
+                <dynamics damping="1.0" friction="0.1"/>
                 <limit effort="2.0" velocity="1.0"/>
             </joint>
