Commit message: Update urdf

File: skratch_description/description/skratch.urdf.xacro (robot description, xacro)
@@ -33,5 +33,5 @@
     </joint>
     <xacro:lidar_mount name="front" parent="skratch_base" >
-        <origin xyz="0.272 -0.16 0.0025" rpy="0.0 0.0 0.0"/>
+        <origin xyz="0.272 -0.168 0.0025" rpy="0.0 0.0 0.0"/>
     </xacro:lidar_mount>
     <xacro:lidar_mount name="back" parent="skratch_base" >

File: skratch_description/description/wheels/kelo_drive.xacro (robot description, xacro)
@@ -30,4 +30,5 @@
             <parent link="${parent}"/>
             <child link="${name}_pivot_link" />
+            <dynamics damping="0.1" friction="0.05"/>
             <limit effort="2.0" velocity="1.0"/>
         </joint>

Commit message: Update names

File: skratch_description/description/skratch.urdf.xacro (robot description, xacro)
@@ -22,14 +22,14 @@
         <child link="skratch_base"/>
     </joint>
-    <xacro:kelo_drive_top_part name="front_left_drive_top_part" parent="skratch_base" drive_name="skratch_1_drive" movable_joints="$(arg movable_joints)">
+    <xacro:kelo_drive_top_part name="front_left" parent="skratch_base" movable_joints="$(arg movable_joints)">
         <origin xyz="0.202 0.118 -0.054" rpy="0.0 0 0.0"/>
     </xacro:kelo_drive_top_part>
-    <xacro:kelo_drive_top_part name="front_right_drive_top_part" parent="skratch_base" drive_name="skratch_2_drive" movable_joints="$(arg movable_joints)">
+    <xacro:kelo_drive_top_part name="front_right" parent="skratch_base" movable_joints="$(arg movable_joints)">
         <origin xyz="0.202 -0.118 -0.054" rpy="0.0 0 0.0"/>
     </xacro:kelo_drive_top_part>
-    <xacro:kelo_drive_top_part name="rear_left_drive_top_part" parent="skratch_base" drive_name="skratch_3_drive" movable_joints="$(arg movable_joints)">
+    <xacro:kelo_drive_top_part name="rear_left" parent="skratch_base" movable_joints="$(arg movable_joints)">
         <origin xyz="-0.202  0.118 -0.054" rpy="0.0 0 0.0"/>
     </xacro:kelo_drive_top_part>
-    <xacro:kelo_drive_top_part name="rear_right_drive_top_part" parent="skratch_base" drive_name="skratch_4_drive" movable_joints="$(arg movable_joints)">
+    <xacro:kelo_drive_top_part name="rear_right" parent="skratch_base" movable_joints="$(arg movable_joints)">
         <origin xyz="-0.202 -0.118 -0.054" rpy="0.0 0 0.0"/>
     </xacro:kelo_drive_top_part>

File: skratch_description/description/wheels/kelo_drive_mid.xacro (robot description, xacro)
@@ -32,5 +32,5 @@
 -->
 <robot xmlns:xacro="http://www.ros.org/wiki/xacro">
-    <xacro:macro name="kelo_drive" params="name parent *origin movable_joints:=true">
+    <xacro:macro name="kelo_drive_mid" params="name parent *origin movable_joints:=true">
         <xacro:include filename="$(find skratch_description)/description/wheels/kelo_drive_wheel.xacro"/>
         <link name="${name}_pivot_link">

File: skratch_description/description/wheels/kelo_drive_top_part.xacro (robot description, xacro)
@@ -8,6 +8,6 @@
 -->
 <robot xmlns:xacro="http://www.ros.org/wiki/xacro">
-    <xacro:macro name="kelo_drive_top_part" params="name parent drive_name:=default_drive_name *origin movable_joints:=true">
-        <xacro:include filename="$(find skratch_description)/description/wheels/kelo_drive.xacro" />
+    <xacro:macro name="kelo_drive_top_part" params="name parent *origin movable_joints:=true">
+        <xacro:include filename="$(find skratch_description)/description/wheels/kelo_drive_mid.xacro" />
         <link name="${name}_drive_top_part">
             <visual>
@@ -37,7 +37,7 @@
             <child link="${name}_drive_top_part"/>
         </joint>
-        <xacro:kelo_drive name="${drive_name}" parent="${name}_drive_top_part" movable_joints="${movable_joints}">
+        <xacro:kelo_drive_mid name="${name}_drive" parent="${name}_drive_top_part" movable_joints="${movable_joints}">
             <origin xyz="0 0 -0.09" rpy="0 0 0.0"/>
-        </xacro:kelo_drive>
+        </xacro:kelo_drive_mid>
     </xacro:macro>
 </robot>
